File: sensor.brd (EAGLE design)
At the start: 16.8 x 16.5 mm, 2 parts

Commit message: Sensor breakout updated
Other:
- outline, holes or cut-outs redrawn
Changed lines of the file:
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@@
 <layer number="27" name="tValues" color="7" fill="1" visible="yes" active="yes"/>
 <layer number="28" name="bValues" color="7" fill="1" visible="yes" active="yes"/>
-<layer number="29" name="tStop" color="7" fill="3" visible="no" active="yes"/>
-<layer number="30" name="bStop" color="7" fill="6" visible="no" active="yes"/>
+<layer number="29" name="tStop" color="7" fill="3" visible="yes" active="yes"/>
+<layer number="30" name="bStop" color="7" fill="6" visible="yes" active="yes"/>
 <layer number="31" name="tCream" color="7" fill="4" visible="no" active="yes"/>
 <layer number="32" name="bCream" color="7" fill="5" visible="no" active="yes"/>
@@
 <board>
 <plain>
-<wire x1="0" y1="0" x2="16.815" y2="0" width="0" layer="20"/>
+<wire x1="0" y1="0" x2="6.35" y2="0" width="0" layer="20"/>
+<wire x1="6.35" y1="0" x2="6.35" y2="0.635" width="0" layer="20"/>
+<wire x1="6.35" y1="0.635" x2="13.335" y2="0.635" width="0" layer="20"/>
+<wire x1="13.335" y1="0.635" x2="13.335" y2="0" width="0" layer="20"/>
+<wire x1="13.335" y1="0" x2="16.815" y2="0" width="0" layer="20"/>
 <wire x1="16.815" y1="0" x2="16.815" y2="16.5" width="0" layer="20"/>
-<wire x1="16.815" y1="16.5" x2="0" y2="16.5" width="0" layer="20"/>
+<wire x1="16.815" y1="16.5" x2="13.335" y2="16.51" width="0" layer="20"/>
+<wire x1="13.335" y1="16.51" x2="13.335" y2="15.875" width="0" layer="20"/>
+<wire x1="13.335" y1="15.875" x2="6.35" y2="15.875" width="0" layer="20"/>
+<wire x1="6.35" y1="15.875" x2="6.35" y2="16.5" width="0" layer="20"/>
+<wire x1="6.35" y1="16.5" x2="0" y2="16.5" width="0" layer="20"/>
 <wire x1="0" y1="16.5" x2="0" y2="0" width="0" layer="20"/>
-<text x="6.35" y="13.97" size="2.1844" layer="22" rot="MR0">+</text>
+<text x="5.08" y="13.97" size="2.1844" layer="22" rot="MR0">+</text>
 <text x="5.08" y="11.43" size="1.016" layer="22" rot="MR0">8</text>
 <text x="15.875" y="11.43" size="1.016" layer="22" rot="MR0">MCK</text>
@@
 <text x="5.715" y="3.81" size="1.016" layer="22" rot="MR0">11</text>
 <text x="16.51" y="4.445" size="1.016" layer="22" rot="MR0">SCK</text>
-<text x="6.985" y="1.27" size="1.016" layer="22" rot="MR0">GND</text>
+<text x="6.35" y="1.27" size="1.016" layer="22" rot="MR0">GND</text>
+<rectangle x1="6.35" y1="13.97" x2="13.335" y2="15.24" layer="1"/>
+<rectangle x1="6.35" y1="13.97" x2="13.335" y2="15.24" layer="29"/>
+<rectangle x1="6.35" y1="13.97" x2="13.335" y2="15.24" layer="16" rot="R180"/>
+<rectangle x1="6.35" y1="13.97" x2="13.335" y2="15.24" layer="30" rot="R180"/>
+<rectangle x1="6.35" y1="1.27" x2="13.335" y2="2.54" layer="1"/>
+<rectangle x1="6.35" y1="1.27" x2="13.335" y2="2.54" layer="29"/>
+<rectangle x1="6.35" y1="1.27" x2="13.335" y2="2.54" layer="16" rot="R180"/>
+<rectangle x1="6.35" y1="1.27" x2="13.335" y2="2.54" layer="30"/>
 </plain>
 <attributes>
@@
 </class>
 </classes>
-<designrules name="oshpark-2layer">
+<designrules name="oshpark-2layer (1)">
 <description language="en">&lt;b&gt;OSH Park Design Rules&lt;/b&gt;
 &lt;p&gt;
